Commit message: Fix Launch Bug, Change Process_Image.cpp

File: my_robot/urdf/my_robot.xacro (robot description, xacro)
@@ -69,5 +69,5 @@
       <origin xyz="0 0 0" rpy="0 1.57 1.57"/>
       <geometry>
-        <cylinder radius="0.1" length="0.05"/>
+        <cylinder radius="0.1" length="0.03"/>
       </geometry>
     </collision>
@@ -75,5 +75,5 @@
       <origin xyz="0 0 0" rpy="0 1.57 1.57"/>
       <geometry>
-        <cylinder radius="0.1" length="0.05"/>
+        <cylinder radius="0.1" length="0.03"/>
       </geometry>
     </visual>
@@ -100,5 +100,5 @@
       <origin xyz="0 0 0" rpy="0 1.57 1.57"/>
       <geometry>
-        <cylinder radius="0.1" length="0.05"/>
+        <cylinder radius="0.1" length="0.03"/>
       </geometry>
     </collision>
@@ -106,5 +106,5 @@
       <origin xyz="0 0 0" rpy="0 1.57 1.57"/>
       <geometry>
-        <cylinder radius="0.1" length="0.05"/>
+        <cylinder radius="0.1" length="0.03"/>
       </geometry>
     </visual>
@@ -183,14 +183,14 @@
   </joint>
   <gazebo reference="left_wheel">
-  <material>Gazebo/Green</material>
+  <material>Gazebo/Blue</material>
   </gazebo>
   <gazebo reference="right_wheel">
-  <material>Gazebo/Green</material>
+  <material>Gazebo/Blue</material>
   </gazebo>
   <gazebo reference="chassis">
-  <material>Gazebo/Red</material>
+  <material>Gazebo/Orange</material>
   </gazebo>
   <gazebo reference="camera">
-  <material>Gazebo/Gold</material>
+  <material>Gazebo/Yellow</material>
   </gazebo>
 </robot>

Commit message: Implement AMCL and Navigation

File: my_robot/urdf/my_robot.xacro (robot description, xacro)
@@ -11,5 +11,5 @@
     <pose>0 0 0.1 0 0 0</pose>
     <inertial>
-      <mass value="15.0"/>
+      <mass value="10.0"/>
       <origin xyz="0.0 0 0" rpy=" 0 0 0"/>
       <inertia
@@ -22,5 +22,5 @@
       <origin xyz="0 0 0" rpy=" 0 0 0"/>
       <geometry>
-        <box size=".4 .2 .1"/>
+        <box size=".4 .2 .076"/>
       </geometry>
     </collision>
@@ -28,29 +28,29 @@
       <origin xyz="0 0 0" rpy=" 0 0 0"/>
       <geometry>
-        <box size=".4 .2 .1"/>
+        <box size=".4 .2 .076"/>
       </geometry>
     </visual>
     <collision name='back_caster_collision'>
-      <origin xyz="-0.15 0 -0.05" rpy=" 0 0 0"/>
-      <geometry>
-        <sphere radius="0.0499"/>
+      <origin xyz="-0.15 0 -0.038" rpy=" 0 0 0"/>
+      <geometry>
+        <sphere radius="0.036"/>
       </geometry>
     </collision>
     <visual name='back_caster_visual'>
-      <origin xyz ="-0.15 0 -0.05" rpy=" 0 0 0"/>
-      <geometry>
-        <sphere radius="0.05"/>
+      <origin xyz ="-0.15 0 -0.038" rpy=" 0 0 0"/>
+      <geometry>
+        <sphere radius="0.036"/>
       </geometry>
     </visual>
     <collision name='front_caster_collision'>
-      <origin xyz="0.15 0 -0.05" rpy=" 0 0 0"/>
-      <geometry>
-        <sphere radius="0.0499"/>
+      <origin xyz="0.15 0 -0.038" rpy=" 0 0 0"/>
+      <geometry>
+        <sphere radius="0.036"/>
       </geometry>
     </collision>
     <visual name='front_caster_visual'>
-      <origin xyz="0.15 0 -0.05" rpy=" 0 0 0"/>
-      <geometry>
-        <sphere radius="0.05"/>
+      <origin xyz="0.15 0 -0.038" rpy=" 0 0 0"/>
+      <geometry>
+        <sphere radius="0.036"/>
       </geometry>
     </visual>
@@ -58,5 +58,5 @@
   <link name="left_wheel">
     <inertial>
-      <mass value="5.0"/>
+      <mass value="1.0"/>
       <origin xyz="0 0 0" rpy="0 1.57 1.57"/>
       <inertia
@@ -69,5 +69,5 @@
       <origin xyz="0 0 0" rpy="0 1.57 1.57"/>
       <geometry>
-        <cylinder radius="0.1" length="0.03"/>
+        <cylinder radius="0.075" length="0.04"/>
       </geometry>
     </collision>
@@ -75,10 +75,10 @@
       <origin xyz="0 0 0" rpy="0 1.57 1.57"/>
       <geometry>
-        <cylinder radius="0.1" length="0.03"/>
+        <cylinder radius="0.075" length="0.04"/>
       </geometry>
     </visual>
   </link>
   <joint name="left_wheel_hinge" type="continuous">
-    <origin xyz="0 0.15 0" rpy="0 0 0" />
+    <origin xyz="0 0.13 0" rpy="0 0 0" />
     <parent link="chassis" />
     <child link="left_wheel" />
@@ -87,7 +87,38 @@
     <dynamics damping="1.0" friction="1.0"/>
   </joint>
+  <!-- <link name="left_wheel_2">
+    <inertial>
+      <mass value="1.0"/>
+      <origin xyz="0 0 0" rpy="0 1.57 1.57"/>
+      <inertia
+          ixx="0.1" ixy="0" ixz="0"
+          iyy="0.1" iyz="0"
+          izz="0.1"
+      />
+    </inertial>
+    <collision name="left_wheel_collision_2">
+      <origin xyz="0 0 0" rpy="0 1.57 1.57"/>
+      <geometry>
+        <cylinder radius="0.075" length="0.04"/>
+      </geometry>
+    </collision>
+    <visual name="left_wheel_visual_2">
+      <origin xyz="0 0 0" rpy="0 1.57 1.57"/>
+      <geometry>
+        <cylinder radius="0.075" length="0.04"/>
+      </geometry>
+    </visual>
+  </link>
+  <joint name="left_wheel_hinge_2" type="continuous">
+    <origin xyz="-0.15 0.13 0" rpy="0 0 0" />
+    <parent link="chassis" />
+    <child link="left_wheel_2" />
+    <axis xyz="0 1 0" rpy="0 0 0"/>
+    <limit effort="10000" velocity="1000"/>
+    <dynamics damping="1.0" friction="1.0"/>
+  </joint> -->
   <link name="right_wheel">
     <inertial>
-      <mass value="5.0"/>
+      <mass value="1.0"/>
       <origin xyz="0 0 0" rpy="0 1.57 1.57"/>
       <inertia
@@ -100,5 +131,5 @@
       <origin xyz="0 0 0" rpy="0 1.57 1.57"/>
       <geometry>
-        <cylinder radius="0.1" length="0.03"/>
+        <cylinder radius="0.075" length="0.04"/>
       </geometry>
     </collision>
@@ -106,10 +137,10 @@
       <origin xyz="0 0 0" rpy="0 1.57 1.57"/>
       <geometry>
-        <cylinder radius="0.1" length="0.03"/>
+        <cylinder radius="0.075" length="0.04"/>
       </geometry>
     </visual>
   </link>
   <joint name="right_wheel_hinge" type="continuous">
-    <origin xyz="0 -0.15 0" rpy="0 0 0" />
+    <origin xyz="0 -0.13 0" rpy="0 0 0" />
     <parent link="chassis" />
     <child link="right_wheel" />
@@ -118,4 +149,35 @@
     <dynamics damping="1.0" friction="1.0"/>
   </joint>
+  <!--<link name="right_wheel_2">
+    <inertial>
+      <mass value="1.0"/>
+      <origin xyz="-0.15 0 0" rpy="0 1.57 1.57"/>
+      <inertia
+          ixx="0.1" ixy="0" ixz="0"
+          iyy="0.1" iyz="0"
+          izz="0.1"
+      />
+    </inertial>
+    <collision name="right_wheel_collision_2">
+      <origin xyz="0 0 0" rpy="0 1.57 1.57"/>
+      <geometry>
+        <cylinder radius="0.075" length="0.04"/>
+      </geometry>
+    </collision>
+    <visual name="right_wheel_visual_2">
+      <origin xyz="0 0 0" rpy="0 1.57 1.57"/>
+      <geometry>
+        <cylinder radius="0.075" length="0.04"/>
+      </geometry>
+    </visual>
+  </link>
+  <joint name="right_wheel_hinge_2" type="continuous">
+    <origin xyz="-0.15 -0.13 0" rpy="0 0 0" />
+    <parent link="chassis" />
+    <child link="right_wheel_2" />
+    <axis xyz="0 1 0" rpy="0 0 0"/>
+    <limit effort="10000" velocity="1000"/>
+    <dynamics damping="1.0" friction="1.0"/>
+  </joint> -->
   <link name="camera">
     <inertial>
